File: KICAD/TLF01_V2/TLF01_V2.kicad_pcb (KiCad board)
At the start: 2 copper layers, 95 x 72 mm, 52 parts, among them J1 ERK_PWR, J2 WAVE_IN, J3 EXT_PWR, J4 TP_GND, J5 CUTOFF, J6 WAVE_OUT, Q1 2SC1815, Q10 2SC1815, Q2 2SC1815, Q3 2SC1815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

Commit message: PCB Design
Parts:
- added G***: LOGO, myfootprint:Silk_PNPN_Manufactory_400dpi, F.Cu at (118.1, 120.7)
- added RV1: 10k/A, Potentiometer_THT:Potentiometer_Alps_RK097_Single_Horizontal, F.Cu at (189.2, 118.1)
- J3: footprint Connector_PinHeader_2.54mm:PinHeader_1x03_P2.54mm_Vertical -> Connector_JST:JST_XH_B3B-XH-A_1x03_P2.50mm_Vertical
- Q1, Q10, Q2, Q3, Q4, Q5, Q6, Q7, Q8, Q9: footprint Package_TO_SOT_THT:TO-92L_Inline -> Package_TO_SOT_THT:TO-92_Inline
- moved J2 49.4 mm to (179.1, 123.2)
- moved J4 44.9 mm to (165.1, 123.2)
- moved J5 8.94 mm to (152.4, 123.2), turned to 270 degrees
- moved RV2 3.57 mm to (189.2, 95.2)
- moved C11 2.92 mm to (176.5, 96.5)
- moved C5 2.71 mm to (153.7, 76.2)
- moved C4 2.71 mm to (143.5, 113.0)
- moved Q10 2.20 mm to (151.9, 104.1)
- moved RV3 1.98 mm to (176.3, 109.2)
- moved R10 1.77 mm to (135.9, 121.9)
- moved R4 1.77 mm to (135.9, 110.5)
- moved R5 1.77 mm to (135.9, 72.4)
- moved C6 1.77 mm to (153.7, 83.8)
- moved C1 1.77 mm to (110.5, 74.9)
- moved C2 1.77 mm to (110.5, 108.0)
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- renumbered RV1 to RV2, RV2 to RV3
Connections:
- J2 pad 1: Net-(C3-Pad2) -> Net-(J2-Pad1)
Routing:
- net +12V: track 1.19 -> 112.4 mm
- net -12V: track 0.00 -> 95.1 mm
- net Net-(C3-Pad2): track 0.00 -> 74.2 mm
- net Net-(C4-Pad1): track 0.00 -> 53.7 mm
- net Net-(C5-Pad2): track 0.00 -> 37.1 mm
- net Net-(C11-Pad2): track 0.00 -> 36.5 mm
- net Net-(Q4-Pad3): track 0.00 -> 34.4 mm
- net Net-(Q3-Pad3): track 0.00 -> 34.4 mm
- net Net-(Q2-Pad3): track 0.00 -> 33.9 mm
- net Net-(Q1-Pad3): track 0.00 -> 27.9 mm
- net Net-(Q10-Pad3): track 0.00 -> 26.9 mm
- net Net-(J2-Pad1): track 0.00 -> 23.2 mm
- net Net-(R12-Pad1): track 0.00 -> 21.9 mm
- net Net-(C5-Pad1): track 0.00 -> 21.2 mm
- net Net-(RV2-Pad1): track 0.00 -> 20.6 mm
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- added copper zone on F.Cu, net (none)
- added copper zone on B.Cu, net GND
Other:
- board text added: "AUDIO_IN"
- board text added: "AUDIO_OUT"
- board text added: "CUTOFF"
- board text added: "G"
- board text added: "GND"
- board text added: "INPUT_LVL"
- board text added: "RESONANCE"
- board text added: "RESONANCE TRIM"
- board text added: "TLF01 V2.0"
- board text added: "V- G V+"
- board text added: "https://dad8893.blogspot.com/"

Commit message: Update PCB Design
Parts:
- J2: value WAVE_IN -> IN
- J6: value WAVE_OUT -> OUT
- moved J2 44.7 mm to (190.5, 80.0), turned to 180 degrees
- moved J4 5.08 mm to (170.2, 123.2)
- moved J6 2.84 mm to (190.5, 72.4)
Routing:
- net Net-(J2-Pad1): track 23.2 -> 36.7 mm
- net Net-(J6-Pad1): track 7.62 -> 9.94 mm
- net (no net): vias 20 -> 0
- added copper zone on F.Cu, net GND
- removed copper zone on F.Cu, net (none)
Other:
- board text added: "IN"
- board text added: "OUT"
- board text removed: "AUDIO_IN"
- board text removed: "AUDIO_OUT"
Changed lines of the file:
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@@
     (thickness 1.6)
     (drawings 17)
-    (tracks 192)
+    (tracks 172)
     (zones 0)
     (modules 54)
@@
     (46 B.CrtYd user)
     (47 F.CrtYd user)
-    (48 B.Fab user hide)
+    (48 B.Fab user)
     (49 F.Fab user hide)
   )
   (setup
-    (last_trace_width 0.75)
+    (last_trace_width 0.25)
     (user_trace_width 0.5)
     (user_trace_width 0.75)
@@
     (solder_mask_min_width 0.25)
     (aux_axis_origin 0 0)
-    (visible_elements 7FFFFFFF)
+    (visible_elements 7FFFF7FF)
     (pcbplotparams
       (layerselection 0x010fc_ffffffff)
@@
   )
   (module Connector_PinHeader_2.54mm:PinHeader_1x02_P2.54mm_Vertical (layer F.Cu)
-    (at 189.23 74.93)
+    (at 190.5 72.39)
     (descr "Through hole straight pin header, 1x02, 2.54mm pitch, single row")
     (tags "Through hole pin header THT 1x02 2.54mm single row")
-    (fp_text reference J6 (at 0 -2.33) (layer F.SilkS)
+    (fp_text reference J6 (at -1.27 -3.81 90) (layer F.SilkS)
       (effects (font (size 1 1) (thickness 0.15)))
     )
-    (fp_text value WAVE_OUT (at 0 4.87) (layer F.Fab)
+    (fp_text value OUT (at 0 4.87) (layer F.Fab)
       (effects (font (size 1 1) (thickness 0.15)))
     )
@@
     (descr "Through hole straight pin header, 1x02, 2.54mm pitch, single row")
     (tags "Through hole pin header THT 1x02 2.54mm single row")
-    (fp_text reference J5 (at 0 -2.33 90) (layer F.SilkS)
+    (fp_text reference J5 (at 0 -3.81 90) (layer F.SilkS)
       (effects (font (size 1 1) (thickness 0.15)))
     )
@@
   )
   (module Connector_PinHeader_2.54mm:PinHeader_1x02_P2.54mm_Vertical (layer F.Cu)
-    (at 165.1 123.19)
+    (at 170.18 123.19)
     (descr "Through hole straight pin header, 1x02, 2.54mm pitch, single row")
     (tags "Through hole pin header THT 1x02 2.54mm single row")
@@
   )
   (module Connector_PinHeader_2.54mm:PinHeader_1x02_P2.54mm_Vertical (layer F.Cu)
-    (at 179.07 123.19 270)
+    (at 190.5 80.01 180)
     (descr "Through hole straight pin header, 1x02, 2.54mm pitch, single row")
     (tags "Through hole pin header THT 1x02 2.54mm single row")
-    (fp_text reference J2 (at 0 -2.33 90) (layer F.SilkS)
+    (fp_text reference J2 (at 1.27 -3.81 90) (layer F.SilkS)
       (effects (font (size 1 1) (thickness 0.15)))
     )
-    (fp_text value WAVE_IN (at 0 4.87 90) (layer F.Fab)
+    (fp_text value IN (at 0 4.87) (layer F.Fab)
       (effects (font (size 1 1) (thickness 0.15)))
     )
@@
     (fp_line (start 1.8 4.35) (end 1.8 -1.8) (layer F.CrtYd) (width 0.05))
     (fp_line (start 1.8 -1.8) (end -1.8 -1.8) (layer F.CrtYd) (width 0.05))
-    (fp_text user %R (at 0 1.27) (layer F.Fab)
+    (fp_text user %R (at 0 1.27 90) (layer F.Fab)
       (effects (font (size 1 1) (thickness 0.15)))
     )
-    (pad 1 thru_hole rect (at 0 0 270) (size 1.7 1.7) (drill 1) (layers *.Cu *.Mask)
+    (pad 1 thru_hole rect (at 0 0 180) (size 1.7 1.7) (drill 1) (layers *.Cu *.Mask)
       (net 31 "Net-(J2-Pad1)"))
-    (pad 2 thru_hole oval (at 0 2.54 270) (size 1.7 1.7) (drill 1) (layers *.Cu *.Mask)
+    (pad 2 thru_hole oval (at 0 2.54 180) (size 1.7 1.7) (drill 1) (layers *.Cu *.Mask)
       (net 1 GND))
     (model ${KISYS3DMOD}/Connector_PinHeader_2.54mm.3dshapes/PinHeader_1x02_P2.54mm_Vertical.wrl
@@
     (effects (font (size 1 1) (thickness 0.15)) (justify left))
   )
-  (gr_text G (at 187.96 80.01 90) (layer F.SilkS)
+  (gr_text G (at 194.31 75.057 90) (layer F.SilkS)
     (effects (font (size 1 1) (thickness 0.15)))
   )
-  (gr_text AUDIO_OUT (at 191.77 76.2 90) (layer F.SilkS)
+  (gr_text OUT (at 191.77 67.945 90) (layer F.SilkS)
     (effects (font (size 1 1) (thickness 0.15)))
   )
@@
     (effects (font (size 1 1) (thickness 0.15)))
   )
-  (gr_text G (at 175.26 120.65) (layer F.SilkS)
+  (gr_text G (at 194.31 77.6478 90) (layer F.SilkS)
     (effects (font (size 1 1) (thickness 0.15)))
   )
-  (gr_text G (at 148.59 120.65) (layer F.SilkS)
+  (gr_text G (at 148.59 119.38) (layer F.SilkS)
     (effects (font (size 1 1) (thickness 0.15)))
   )
-  (gr_text CUTOFF (at 151.13 125.73) (layer F.SilkS)
+  (gr_text CUTOFF (at 151.13 128.27) (layer F.SilkS)
     (effects (font (size 1 1) (thickness 0.15)))
   )
-  (gr_text AUDIO_IN (at 177.8 125.73) (layer F.SilkS)
+  (gr_text IN (at 191.77 83.82 90) (layer F.SilkS)
     (effects (font (size 1 1) (thickness 0.15)))
   )
@@
   (gr_line (start 100 60) (end 195 60) (layer Edge.Cuts) (width 0.05))
   (gr_line (start 100 132) (end 100 60) (layer Edge.Cuts) (width 0.05))
-  (via (at 111.76 114.3) (size 0.8) (drill 0.4) (layers F.Cu B.Cu) (net 0))
-  (via (at 116.84 114.3) (size 0.8) (drill 0.4) (layers F.Cu B.Cu) (net 0))
-  (via (at 116.84 63.5) (size 0.8) (drill 0.4) (layers F.Cu B.Cu) (net 0))
-  (via (at 121.92 63.5) (size 0.8) (drill 0.4) (layers F.Cu B.Cu) (net 0))
-  (via (at 127 63.5) (size 0.8) (drill 0.4) (layers F.Cu B.Cu) (net 0))
-  (via (at 116.84 68.58) (size 0.8) (drill 0.4) (layers F.Cu B.Cu) (net 0))
-  (via (at 121.92 68.58) (size 0.8) (drill 0.4) (layers F.Cu B.Cu) (net 0))
-  (via (at 119.38 71.12) (size 0.8) (drill 0.4) (layers F.Cu B.Cu) (net 0))
-  (via (at 119.38 66.04) (size 0.8) (drill 0.4) (layers F.Cu B.Cu) (net 0))
-  (via (at 124.46 66.04) (size 0.8) (drill 0.4) (layers F.Cu B.Cu) (net 0))
-  (via (at 114.3 66.04) (size 0.8) (drill 0.4) (layers F.Cu B.Cu) (net 0))
-  (via (at 111.76 63.5) (size 0.8) (drill 0.4) (layers F.Cu B.Cu) (net 0))
-  (via (at 190.5 101.6) (size 0.8) (drill 0.4) (layers F.Cu B.Cu) (net 0))
-  (via (at 190.5 106.68) (size 0.8) (drill 0.4) (layers F.Cu B.Cu) (net 0))
-  (via (at 187.96 104.14) (size 0.8) (drill 0.4) (layers F.Cu B.Cu) (net 0))
-  (via (at 114.3 111.76) (size 0.8) (drill 0.4) (layers F.Cu B.Cu) (net 0))
-  (via (at 116.84 109.22) (size 0.8) (drill 0.4) (layers F.Cu B.Cu) (net 0))
-  (via (at 119.38 111.76) (size 0.8) (drill 0.4) (layers F.Cu B.Cu) (net 0))
-  (via (at 121.92 114.3) (size 0.8) (drill 0.4) (layers F.Cu B.Cu) (net 0))
-  (via (at 121.92 109.22) (size 0.8) (drill 0.4) (layers F.Cu B.Cu) (net 0))
   (segment (start 184.11 72.35) (end 184.15 72.39) (width 0.75) (layer F.Cu) (net 2) (status 30))
   (segment (start 184.11 68.58) (end 184.11 72.35) (width 0.75) (layer B.Cu) (net 2) (status 30))
@@
   (segment (start 152.4 118.11) (end 152.4 123.19) (width 0.75) (layer F.Cu) (net 19) (status 30))
   (segment (start 184.15 74.93) (end 184.15 77.47) (width 0.75) (layer F.Cu) (net 20) (status 30))
-  (segment (start 184.15 74.93) (end 189.23 74.93) (width 0.75) (layer F.Cu) (net 20) (status 30))
+  (segment (start 184.15 74.93) (end 185.42 74.93) (width 0.75) (layer F.Cu) (net 20))
+  (segment (start 185.42 74.93) (end 187.96 72.39) (width 0.75) (layer F.Cu) (net 20))
+  (segment (start 187.96 72.39) (end 190.5 72.39) (width 0.75) (layer F.Cu) (net 20))
   (segment (start 160.02 72.39) (end 140.97 72.39) (width 0.75) (layer F.Cu) (net 21) (status 30))
   (segment (start 140.97 72.39) (end 135.89 72.39) (width 0.75) (layer F.Cu) (net 21) (status 30))
@@
   (segment (start 173.736 111.76) (end 176.276 109.22) (width 0.75) (layer F.Cu) (net 30) (status 20))
   (segment (start 163.83 111.76) (end 173.736 111.76) (width 0.75) (layer F.Cu) (net 30) (status 10))
-  (segment (start 179.07 123.19) (end 189.23 123.19) (width 0.75) (layer F.Cu) (net 31))
-  (segment (start 189.23 123.19) (end 191.77 120.65) (width 0.75) (layer F.Cu) (net 31))
-  (segment (start 191.77 120.65) (end 191.77 114.3) (width 0.75) (layer F.Cu) (net 31))
-  (segment (start 191.77 114.3) (end 190.5 113.03) (width 0.75) (layer F.Cu) (net 31))
-  (segment (start 190.42 113.11) (end 189.23 113.11) (width 0.75) (layer F.Cu) (net 31))
-  (segment (start 190.5 113.03) (end 190.42 113.11) (width 0.75) (layer F.Cu) (net 31))
+  (segment (start 193.04 109.3) (end 189.23 113.11) (width 0.75) (layer F.Cu) (net 31))
+  (segment (start 193.04 80.95) (end 193.04 109.3) (width 0.75) (layer F.Cu) (net 31))
+  (segment (start 190.5 80.01) (end 192.1 80.01) (width 0.75) (layer F.Cu) (net 31))
+  (segment (start 192.1 80.01) (end 193.04 80.95) (width 0.75) (layer F.Cu) (net 31))
   (segment (start 189.23 97.79) (end 189.23 95.25) (width 0.75) (layer F.Cu) (net 32) (status 20))
   (segment (start 176.276 104.14) (end 182.88 104.14) (width 0.75) (layer F.Cu) (net 32) (status 10))
@@
     )
   )
-  (zone (net 0) (net_name "") (layer F.Cu) (hatch edge 0.508)
+  (zone (net 1) (net_name GND) (layer F.Cu) (hatch edge 0.508)
     (connect_pads (clearance 0.508))
     (min_thickness 0.254)
