File: KICAD/TLF01_V2/TLF01_V2.sch (KiCad schematic (older format))
At the start: 52 parts, among them J1 ERK_PWR, J2 WAVE_IN, J3 EXT_PWR, J4 TP_GND, J5 CUTOFF, J6 WAVE_OUT, Q1 2SC1815, Q10 2SC1815, Q2 2SC1815, Q3 2SC1815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

Commit message: PCB Design
Parts:
- added RV1: 10k/A, Potentiometer_THT:Potentiometer_Alps_RK097_Single_Horizontal, symbol Device:R_POT
- J3: footprint Connector_PinHeader_2.54mm:PinHeader_1x03_P2.54mm_Vertical -> Connector_JST:JST_XH_B3B-XH-A_1x03_P2.50mm_Vertical
- Q1, Q10, Q2, Q3, Q4, Q5, Q6, Q7, Q8, Q9: footprint Package_TO_SOT_THT:TO-92L_Inline -> Package_TO_SOT_THT:TO-92_Inline
- renumbered RV1 to RV2, RV2 to RV3
Connections:
- net GND: now also RV1.1
- net at C3.2: now also RV1.2; no longer J2.1 (Pin_1)
- new net: J2.1 (Pin_1), RV1.3
Other:
- moved on the sheet: C3, J2
Changed lines of the file:
@@
 EESchema Schematic File Version 4
+LIBS:TLF01_V2-cache
 EELAYER 30 0
 EELAYER END
@@
 Sheet 1 1
 Title "TLF01_V2"
-Date "2020-05-03"
+Date "2020-05-05"
 Rev "Ver. 2.0"
 Comp "PNPN Manufactory"
@@
 F 0 "Q1" H 5440 1746 50  0000 L CNN
 F 1 "2SC1815" H 5440 1655 50  0000 L CNN
-F 2 "Package_TO_SOT_THT:TO-92L_Inline" H 5450 1800 50  0001 C CNN
+F 2 "Package_TO_SOT_THT:TO-92_Inline" H 5450 1800 50  0001 C CNN
 F 3 "~" H 5250 1700 50  0001 C CNN
 	1    5250 1700
@@
 F 0 "Q2" H 5440 2896 50  0000 L CNN
 F 1 "2SC1815" H 5440 2805 50  0000 L CNN
-F 2 "Package_TO_SOT_THT:TO-92L_Inline" H 5450 2950 50  0001 C CNN
+F 2 "Package_TO_SOT_THT:TO-92_Inline" H 5450 2950 50  0001 C CNN
 F 3 "~" H 5250 2850 50  0001 C CNN
 	1    5250 2850
@@
 F 0 "Q6" H 6840 1746 50  0000 L CNN
 F 1 "2SC1815" H 6840 1655 50  0000 L CNN
-F 2 "Package_TO_SOT_THT:TO-92L_Inline" H 6850 1800 50  0001 C CNN
+F 2 "Package_TO_SOT_THT:TO-92_Inline" H 6850 1800 50  0001 C CNN
 F 3 "~" H 6650 1700 50  0001 C CNN
 	1    6650 1700
@@
 F 0 "Q7" H 6840 2896 50  0000 L CNN
 F 1 "2SC1815" H 6840 2805 50  0000 L CNN
-F 2 "Package_TO_SOT_THT:TO-92L_Inline" H 6850 2950 50  0001 C CNN
+F 2 "Package_TO_SOT_THT:TO-92_Inline" H 6850 2950 50  0001 C CNN
 F 3 "~" H 6650 2850 50  0001 C CNN
 	1    6650 2850
@@
 F 0 "Q3" H 5440 3746 50  0000 L CNN
 F 1 "2SC1815" H 5440 3655 50  0000 L CNN
-F 2 "Package_TO_SOT_THT:TO-92L_Inline" H 5450 3800 50  0001 C CNN
+F 2 "Package_TO_SOT_THT:TO-92_Inline" H 5450 3800 50  0001 C CNN
 F 3 "~" H 5250 3700 50  0001 C CNN
 	1    5250 3700
@@
 F 0 "Q8" H 6840 3746 50  0000 L CNN
 F 1 "2SC1815" H 6840 3655 50  0000 L CNN
-F 2 "Package_TO_SOT_THT:TO-92L_Inline" H 6850 3800 50  0001 C CNN
+F 2 "Package_TO_SOT_THT:TO-92_Inline" H 6850 3800 50  0001 C CNN
 F 3 "~" H 6650 3700 50  0001 C CNN
 	1    6650 3700
@@
 F 0 "Q4" H 5440 4596 50  0000 L CNN
 F 1 "2SC1815" H 5440 4505 50  0000 L CNN
-F 2 "Package_TO_SOT_THT:TO-92L_Inline" H 5450 4650 50  0001 C CNN
+F 2 "Package_TO_SOT_THT:TO-92_Inline" H 5450 4650 50  0001 C CNN
 F 3 "~" H 5250 4550 50  0001 C CNN
 	1    5250 4550
@@
 F 0 "Q9" H 6840 4596 50  0000 L CNN
 F 1 "2SC1815" H 6840 4505 50  0000 L CNN
-F 2 "Package_TO_SOT_THT:TO-92L_Inline" H 6850 4650 50  0001 C CNN
+F 2 "Package_TO_SOT_THT:TO-92_Inline" H 6850 4650 50  0001 C CNN
 F 3 "~" H 6650 4550 50  0001 C CNN
 	1    6650 4550
@@
 F 0 "Q5" H 5440 5496 50  0000 L CNN
 F 1 "2SC1815" H 5440 5405 50  0000 L CNN
-F 2 "Package_TO_SOT_THT:TO-92L_Inline" H 5450 5550 50  0001 C CNN
+F 2 "Package_TO_SOT_THT:TO-92_Inline" H 5450 5550 50  0001 C CNN
 F 3 "~" H 5250 5450 50  0001 C CNN
 	1    5250 5450
@@
 F 0 "Q10" H 6840 5496 50  0000 L CNN
 F 1 "2SC1815" H 6840 5405 50  0000 L CNN
-F 2 "Package_TO_SOT_THT:TO-92L_Inline" H 6850 5550 50  0001 C CNN
+F 2 "Package_TO_SOT_THT:TO-92_Inline" H 6850 5550 50  0001 C CNN
 F 3 "~" H 6650 5450 50  0001 C CNN
 	1    6650 5450
@@
 $EndComp
 $Comp
-L Device:R_POT RV1
+L Device:R_POT RV2
 U 1 1 5EB55945
 P 8700 4300
-F 0 "RV1" H 8630 4254 50  0000 R CNN
+F 0 "RV2" H 8630 4254 50  0000 R CNN
 F 1 "50k/B" H 8630 4345 50  0000 R CNN
 F 2 "Potentiometer_THT:Potentiometer_Alps_RK097_Single_Horizontal" H 8700 4300 50  0001 C CNN
@@
 $EndComp
 $Comp
-L Device:R_POT_TRIM RV2
+L Device:R_POT_TRIM RV3
 U 1 1 5EB5417A
 P 8700 5450
-F 0 "RV2" H 8630 5404 50  0000 R CNN
+F 0 "RV3" H 8630 5404 50  0000 R CNN
 F 1 "1k" H 8630 5495 50  0000 R CNN
 F 2 "Potentiometer_THT:Potentiometer_Bourns_3386P_Vertical" H 8700 5450 50  0001 C CNN
@@
 $EndComp
 $Comp
-L power:GND #PWR015
+L power:GND #PWR016
 U 1 1 5EB59381
 P 8300 2100
-F 0 "#PWR015" H 8300 1850 50  0001 C CNN
+F 0 "#PWR016" H 8300 1850 50  0001 C CNN
 F 1 "GND" V 8305 1972 50  0000 R CNN
 F 2 "" H 8300 2100 50  0001 C CNN
@@
 $EndComp
 $Comp
-L power:GND #PWR016
+L power:GND #PWR017
 U 1 1 5EB59CDA
 P 8300 2800
-F 0 "#PWR016" H 8300 2550 50  0001 C CNN
+F 0 "#PWR017" H 8300 2550 50  0001 C CNN
 F 1 "GND" V 8305 2672 50  0000 R CNN
 F 2 "" H 8300 2800 50  0001 C CNN
@@
 	7500 2550 7350 2550
 $Comp
-L power:GND #PWR012
+L power:GND #PWR013
 U 1 1 5EB68AB6
 P 7500 3100
-F 0 "#PWR012" H 7500 2850 50  0001 C CNN
+F 0 "#PWR013" H 7500 2850 50  0001 C CNN
 F 1 "GND" H 7505 2927 50  0000 C CNN
 F 2 "" H 7500 3100 50  0001 C CNN
@@
 L Device:CP C3
 U 1 1 5EB9EB37
-P 3300 5450
-F 0 "C3" V 3045 5450 50  0000 C CNN
-F 1 "10u" V 3136 5450 50  0000 C CNN
-F 2 "Capacitor_THT:CP_Radial_D6.3mm_P2.50mm" H 3338 5300 50  0001 C CNN
-F 3 "~" H 3300 5450 50  0001 C CNN
-	1    3300 5450
+P 3350 5450
+F 0 "C3" V 3095 5450 50  0000 C CNN
+F 1 "10u" V 3186 5450 50  0000 C CNN
+F 2 "Capacitor_THT:CP_Radial_D6.3mm_P2.50mm" H 3388 5300 50  0001 C CNN
+F 3 "~" H 3350 5450 50  0001 C CNN
+	1    3350 5450
 	0    1    1    0
 $EndComp
@@
 $EndComp
 $Comp
-L power:GND #PWR011
+L power:GND #PWR012
 U 1 1 5EBC0763
 P 5950 7100
-F 0 "#PWR011" H 5950 6850 50  0001 C CNN
+F 0 "#PWR012" H 5950 6850 50  0001 C CNN
 F 1 "GND" H 5955 6927 50  0000 C CNN
 F 2 "" H 5950 7100 50  0001 C CNN
@@
 	4150 5450 5050 5450
 Wire Wire Line
-	3600 5450 3450 5450
+	3600 5450 3500 5450
 $Comp
 L Connector_Generic:Conn_01x02 J2
 U 1 1 5EBFB71D
-P 2750 5450
-F 0 "J2" H 2668 5667 50  0000 C CNN
-F 1 "WAVE_IN" H 2668 5576 50  0000 C CNN
-F 2 "Connector_PinHeader_2.54mm:PinHeader_1x02_P2.54mm_Vertical" H 2750 5450 50  0001 C CNN
-F 3 "~" H 2750 5450 50  0001 C CNN
-	1    2750 5450
+P 2150 5200
+F 0 "J2" H 2068 5417 50  0000 C CNN
+F 1 "WAVE_IN" H 2068 5326 50  0000 C CNN
+F 2 "Connector_PinHeader_2.54mm:PinHeader_1x02_P2.54mm_Vertical" H 2150 5200 50  0001 C CNN
+F 3 "~" H 2150 5200 50  0001 C CNN
+	1    2150 5200
 	-1   0    0    -1
 $EndComp
-Wire Wire Line
-	2950 5450 3150 5450
-$Comp
-L power:GND #PWR07
+$Comp
+L power:GND #PWR06
 U 1 1 5EC00F0C
-P 3050 5750
-F 0 "#PWR07" H 3050 5500 50  0001 C CNN
-F 1 "GND" H 3055 5577 50  0000 C CNN
-F 2 "" H 3050 5750 50  0001 C CNN
-F 3 "" H 3050 5750 50  0001 C CNN
-	1    3050 5750
-	1    0    0    -1
-$EndComp
-Wire Wire Line
-	2950 5550 3050 5550
-Wire Wire Line
-	3050 5550 3050 5750
-$Comp
-L power:GND #PWR010
+P 2450 5650
+F 0 "#PWR06" H 2450 5400 50  0001 C CNN
+F 1 "GND" H 2455 5477 50  0000 C CNN
+F 2 "" H 2450 5650 50  0001 C CNN
+F 3 "" H 2450 5650 50  0001 C CNN
+	1    2450 5650
+	1    0    0    -1
+$EndComp
+Wire Wire Line
+	2350 5300 2450 5300
+Wire Wire Line
+	2450 5300 2450 5650
+$Comp
+L power:GND #PWR011
 U 1 1 5EC0A993
 P 4600 7100
-F 0 "#PWR010" H 4600 6850 50  0001 C CNN
+F 0 "#PWR011" H 4600 6850 50  0001 C CNN
 F 1 "GND" H 4605 6927 50  0000 C CNN
 F 2 "" H 4600 7100 50  0001 C CNN
@@
 Connection ~ 9700 2550
 $Comp
-L power:GND #PWR017
+L power:GND #PWR018
 U 1 1 5EC2DE0C
 P 9950 2950
-F 0 "#PWR017" H 9950 2700 50  0001 C CNN
+F 0 "#PWR018" H 9950 2700 50  0001 C CNN
 F 1 "GND" H 9955 2777 50  0000 C CNN
 F 2 "" H 9950 2950 50  0001 C CNN
@@
 	9950 2650 10050 2650
 $Comp
-L power:+12V #PWR013
+L power:+12V #PWR014
 U 1 1 5EC60FCD
 P 7950 2050
-F 0 "#PWR013" H 7950 1900 50  0001 C CNN
+F 0 "#PWR014" H 7950 1900 50  0001 C CNN
 F 1 "+12V" H 7965 2223 50  0000 C CNN
 F 2 "" H 7950 2050 50  0001 C CNN
@@
 $EndComp
 $Comp
-L power:-12V #PWR014
+L power:-12V #PWR015
 U 1 1 5EC61B61
 P 7950 2850
-F 0 "#PWR014" H 7950 2950 50  0001 C CNN
+F 0 "#PWR015" H 7950 2950 50  0001 C CNN
 F 1 "-12V" H 7965 3023 50  0000 C CNN
 F 2 "" H 7950 2850 50  0001 C CNN
@@
 Connection ~ 7950 2800
 $Comp
-L power:+12V #PWR09
+L power:+12V #PWR010
 U 1 1 5EC71FCA
 P 4600 850
-F 0 "#PWR09" H 4600 700 50  0001 C CNN
+F 0 "#PWR010" H 4600 700 50  0001 C CNN
 F 1 "+12V" H 4615 1023 50  0000 C CNN
 F 2 "" H 4600 850 50  0001 C CNN
@@
 F 0 "J3" H 3580 1992 50  0000 L CNN
 F 1 "EXT_PWR" H 3580 1901 50  0000 L CNN
-F 2 "Connector_PinHeader_2.54mm:PinHeader_1x03_P2.54mm_Vertical" H 3500 1950 50  0001 C CNN
+F 2 "Connector_JST:JST_XH_B3B-XH-A_1x03_P2.50mm_Vertical" H 3500 1950 50  0001 C CNN
 F 3 "~" H 3500 1950 50  0001 C CNN
 	1    3500 1950
@@
 Connection ~ 3200 3200
 $Comp
-L power:GND #PWR08
+L power:GND #PWR09
 U 1 1 5ED5EC56
 P 3200 3350
-F 0 "#PWR08" H 3200 3100 50  0001 C CNN
+F 0 "#PWR09" H 3200 3100 50  0001 C CNN
 F 1 "GND" H 3205 3177 50  0000 C CNN
 F 2 "" H 3200 3350 50  0001 C CNN
@@
 $EndComp
 $Comp
-L power:-12V #PWR06
+L power:-12V #PWR07
 U 1 1 5EDA3473
 P 2750 4400
-F 0 "#PWR06" H 2750 4500 50  0001 C CNN
+F 0 "#PWR07" H 2750 4500 50  0001 C CNN
 F 1 "-12V" H 2765 4573 50  0000 C CNN
 F 2 "" H 2750 4400 50  0001 C CNN
@@
 	1    0    0    -1
 $EndComp
+$Comp
+L Device:R_POT RV1
+U 1 1 5EB21873
+P 2900 5450
+F 0 "RV1" H 2830 5404 50  0000 R CNN
+F 1 "10k/A" H 2830 5495 50  0000 R CNN
+F 2 "Potentiometer_THT:Potentiometer_Alps_RK097_Single_Horizontal" H 2900 5450 50  0001 C CNN
+F 3 "~" H 2900 5450 50  0001 C CNN
+	1    2900 5450
+	1    0    0    1
+$EndComp
+$Comp
+L power:GND #PWR08
+U 1 1 5EB4FC53
+P 2900 5650
+F 0 "#PWR08" H 2900 5400 50  0001 C CNN
+F 1 "GND" H 2905 5477 50  0000 C CNN
+F 2 "" H 2900 5650 50  0001 C CNN
+F 3 "" H 2900 5650 50  0001 C CNN
+	1    2900 5650
+	1    0    0    -1
+$EndComp
+Wire Wire Line
+	2900 5600 2900 5650
+Wire Wire Line
+	2350 5200 2900 5200
+Wire Wire Line
+	2900 5200 2900 5300
+Wire Wire Line
+	3050 5450 3200 5450
 $EndSCHEMATC

Commit message: Update PCB Design
Parts:
- J2: value WAVE_IN -> AUDIO_IN
- J6: value WAVE_OUT -> AUDIO_OUT
Changed lines of the file:
@@
 P 2150 5200
 F 0 "J2" H 2068 5417 50  0000 C CNN
-F 1 "WAVE_IN" H 2068 5326 50  0000 C CNN
+F 1 "AUDIO_IN" H 2068 5326 50  0000 C CNN
 F 2 "Connector_PinHeader_2.54mm:PinHeader_1x02_P2.54mm_Vertical" H 2150 5200 50  0001 C CNN
 F 3 "~" H 2150 5200 50  0001 C CNN
@@
 P 10250 2550
 F 0 "J6" H 10330 2542 50  0000 L CNN
-F 1 "WAVE_OUT" H 10330 2451 50  0000 L CNN
+F 1 "AUDIO_OUT" H 10330 2451 50  0000 L CNN
 F 2 "Connector_PinHeader_2.54mm:PinHeader_1x02_P2.54mm_Vertical" H 10250 2550 50  0001 C CNN
 F 3 "~" H 10250 2550 50  0001 C CNN
