File: KICAD/TLF01_V2_rev_A/TLF01_V2.kicad_pcb (KiCad board)
At the start: 2 copper layers, 95 x 72 mm, 54 parts, among them J1 ERK_PWR, J2 AUDIO_IN, J3 EXT_PWR, J4 TP_GND, J5 CUTOFF, J6 AUDIO_OUT, Q1 2SC1815, Q10 2SC1815, Q2 2SC1815, Q3 2SC1815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

Commit message: Update: PCB Design
Parts:
- J2, J5, J6: footprint Connector_PinHeader_2.54mm:PinHeader_1x02_P2.54mm_Vertical -> Connector_JST:JST_XH_B2B-XH-A_1x02_P2.50mm_Vertical
- moved D1 14.0 mm to (124.5, 66.0), turned to 90 degrees
- moved D2 12.7 mm to (124.5, 99.1), turned to 90 degrees
- moved R2 12.7 mm to (119.4, 94.0)
- moved R1 12.7 mm to (119.4, 61.0)
- moved C1 6.48 mm to (132.1, 69.8)
- moved C2 6.48 mm to (132.1, 95.2)
- moved RV3 5.26 mm to (189.2, 96.5), turned to 180 degrees
- moved G*** 5.08 mm to (157.5, 43.2)
- moved J3 3.81 mm to (132.1, 78.7)
- moved R9 3.10 mm to (139.7, 83.8)
- moved R5 2.84 mm to (147.3, 57.1)
- moved R6 2.84 mm to (139.7, 61.0)
- moved R11 2.72 mm to (162.6, 102.9)
- moved J5 2.56 mm to (162.6, 116.8), turned to 180 degrees
- moved C3 2.54 mm to (139.7, 97.8)
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Other:
- board text added: "TLF01 V2.0 rev.A"
- board text removed: "TLF01 V2.0"

Commit message: Update: PCB Design
Parts:
- removed J6: AUDIO_OUT, Connector_JST:JST_XH_B2B-XH-A_1x02_P2.50mm_Vertical
- J2: value AUDIO_IN -> Audio_In_Out; footprint Connector_JST:JST_XH_B2B-XH-A_1x02_P2.50mm_Vertical -> Connector_JST:JST_XH_B4B-XH-A_1x04_P2.50mm_Vertical
- moved G*** 88.2 mm to (113.0, 119.4)
- moved R12 20.5 mm to (167.6, 77.5)
- moved R16 20.5 mm to (167.6, 66.0)
- moved Q6 20.5 mm to (154.9, 69.8)
- moved Q7 20.5 mm to (154.9, 78.7)
- moved Q8 20.5 mm to (154.9, 87.6)
- moved Q9 20.5 mm to (154.9, 96.5)
- moved R14 20.5 mm to (160.0, 69.8)
- moved R13 20.5 mm to (160.0, 73.7)
- moved C10 19.7 mm to (173.9, 77.5)
- moved C9 19.7 mm to (176.6, 62.2)
- moved U1 19.7 mm to (171.4, 66.0)
- moved C1 19.3 mm to (114.3, 77.5)
- moved C2 19.3 mm to (114.3, 102.9)
- moved J3 19.3 mm to (114.3, 86.4)
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Connections:
- J2 pad 1: Net-(J2-Pad1) -> Audio_Out
- RV1 pad 3: Net-(J2-Pad1) -> Net-(J2-Pad3)
- U1 pad 6: Net-(J6-Pad1) -> Audio_Out
- U1 pad 7: Net-(J6-Pad1) -> Audio_Out
Routing:
- net +12V: track 0.00 -> 113.7 mm
- net -12V: track 0.00 -> 110.9 mm
- net Net-(C3-Pad2): track 0.00 -> 71.9 mm
- net Net-(C4-Pad1): track 0.00 -> 47.9 mm
- net Net-(Q4-Pad3): track 0.00 -> 37.4 mm
- net Net-(Q3-Pad3): track 0.00 -> 37.4 mm
- net Net-(J2-Pad3): track 0.00 -> 37.3 mm
- net Net-(C11-Pad2): track 0.00 -> 35.8 mm
- net Net-(Q2-Pad3): track 0.00 -> 35.1 mm
- net Net-(C5-Pad2): track 0.00 -> 35.0 mm
- net Net-(Q1-Pad3): track 0.00 -> 29.2 mm
- net Net-(R12-Pad1): track 0.00 -> 27.2 mm
- net Net-(RV2-Pad1): track 0.00 -> 22.7 mm
- net Net-(C5-Pad1): track 0.00 -> 21.7 mm
- net Net-(Q10-Pad3): track 0.00 -> 21.6 mm
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- added copper zone on B.Cu, net GND
- added copper zone on F.Cu, net GND
Other:
- board text added: "CUTOFF"
- board text added: "GND"
- board text added: "https://dad8893.blogspot.com/"

Commit message: Update: PCB Design
Connections:
- J2 pad 3: Net-(J2-Pad3) -> GND
- J2 pad 4: GND -> Net-(J2-Pad4)
- RV1 pad 3: Net-(J2-Pad3) -> Net-(J2-Pad4)
Routing:
- net Net-(J2-Pad3): track 37.3 -> 0.00 mm
- net Net-(J2-Pad4): track 0.00 -> 34.1 mm
