File: KICAD/TLF01_V2_rev_A/TLF01_V2.sch (KiCad schematic (older format))
At the start: 53 parts, among them J1 ERK_PWR, J2 AUDIO_IN, J3 EXT_PWR, J4 TP_GND, J5 CUTOFF, J6 AUDIO_OUT, Q1 2SC1815, Q10 2SC1815, Q2 2SC1815, Q3 2SC1815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

Commit message: Update: PCB Design
Parts:
- removed J2: AUDIO_IN, Connector_PinHeader_2.54mm:PinHeader_1x02_P2.54mm_Vertical, symbol Connector_Generic:Conn_01x02
- removed J6: AUDIO_OUT, Connector_PinHeader_2.54mm:PinHeader_1x02_P2.54mm_Vertical, symbol Connector_Generic:Conn_01x02
- added J2: Audio_In_Out, Connector_JST:JST_XH_B4B-XH-A_1x04_P2.50mm_Vertical, symbol Connector_Generic:Conn_01x04
- J5: footprint Connector_PinHeader_2.54mm:PinHeader_1x02_P2.54mm_Vertical -> Connector_JST:JST_XH_B2B-XH-A_1x02_P2.50mm_Vertical
Connections:
- net GND: now also J2.2 (Pin_2), J2.4 (Pin_4)
- net at RV1.3: now also J2.1 (Pin_1)
- net Audio_Out: now reaches U1.6 (-), U1.7
- net Audio_Out: now also J2.3 (Pin_3)
Changed lines of the file:
@@
 Sheet 1 1
 Title "TLF01_V2"
-Date "2020-08-16"
+Date "2020-08-17"
 Rev "A"
 Comp "PNPN Manufactory"
@@
 F 0 "J5" H 5980 6842 50  0000 L CNN
 F 1 "CUTOFF" H 5980 6751 50  0000 L CNN
-F 2 "Connector_PinHeader_2.54mm:PinHeader_1x02_P2.54mm_Vertical" H 5900 6850 50  0001 C CNN
+F 2 "Connector_JST:JST_XH_B2B-XH-A_1x02_P2.50mm_Vertical" H 5900 6850 50  0001 C CNN
 F 3 "~" H 5900 6850 50  0001 C CNN
 	1    5900 6850
@@
 	3300 5500 3200 5500
 $Comp
-L Connector_Generic:Conn_01x02 J2
-U 1 1 5EBFB71D
-P 1850 5250
-F 0 "J2" H 1768 5467 50  0000 C CNN
-F 1 "AUDIO_IN" H 1768 5376 50  0000 C CNN
-F 2 "Connector_PinHeader_2.54mm:PinHeader_1x02_P2.54mm_Vertical" H 1850 5250 50  0001 C CNN
-F 3 "~" H 1850 5250 50  0001 C CNN
-	1    1850 5250
-	-1   0    0    -1
-$EndComp
-$Comp
 L power:GND #PWR06
 U 1 1 5EC00F0C
-P 2150 5700
-F 0 "#PWR06" H 2150 5450 50  0001 C CNN
-F 1 "GND" H 2155 5527 50  0000 C CNN
-F 2 "" H 2150 5700 50  0001 C CNN
-F 3 "" H 2150 5700 50  0001 C CNN
-	1    2150 5700
-	1    0    0    -1
-$EndComp
-Wire Wire Line
-	2050 5350 2150 5350
-Wire Wire Line
-	2150 5350 2150 5700
+P 2200 5700
+F 0 "#PWR06" H 2200 5450 50  0001 C CNN
+F 1 "GND" H 2205 5527 50  0000 C CNN
+F 2 "" H 2200 5700 50  0001 C CNN
+F 3 "" H 2200 5700 50  0001 C CNN
+	1    2200 5700
+	1    0    0    -1
+$EndComp
+Wire Wire Line
+	2200 5350 2200 5550
 $Comp
 L power:GND #PWR011
@@
 	4300 7150 4300 6850
 Connection ~ 4300 6850
-$Comp
-L Connector_Generic:Conn_01x02 J6
-U 1 1 5EC28907
-P 9700 2400
-F 0 "J6" H 9780 2392 50  0000 L CNN
-F 1 "AUDIO_OUT" H 9780 2301 50  0000 L CNN
-F 2 "Connector_PinHeader_2.54mm:PinHeader_1x02_P2.54mm_Vertical" H 9700 2400 50  0001 C CNN
-F 3 "~" H 9700 2400 50  0001 C CNN
-	1    9700 2400
-	1    0    0    -1
-$EndComp
-$Comp
-L power:GND #PWR018
-U 1 1 5EC2DE0C
-P 9400 2800
-F 0 "#PWR018" H 9400 2550 50  0001 C CNN
-F 1 "GND" H 9405 2627 50  0000 C CNN
-F 2 "" H 9400 2800 50  0001 C CNN
-F 3 "" H 9400 2800 50  0001 C CNN
-	1    9400 2800
-	1    0    0    -1
-$EndComp
-Wire Wire Line
-	9400 2800 9400 2500
-Wire Wire Line
-	9400 2500 9500 2500
 $Comp
 L power:+12V #PWR014
@@
 	1    0    0    1
 $EndComp
-Text Notes 2000 6800 0    100  ~ 0
+Text Notes 1750 6700 0    100  ~ 0
 C&T: Cut & Try
 $Comp
@@
 	2600 5650 2600 5700
 Wire Wire Line
-	2050 5250 2600 5250
-Wire Wire Line
 	2600 5250 2600 5350
 Wire Wire Line
@@
 	9350 2000 9350 2400
 Connection ~ 9350 2400
+Text GLabel 9500 2400 2    59   Output ~ 0
+Audio_Out
 Wire Wire Line
 	9350 2400 9500 2400
+$Comp
+L Connector_Generic:Conn_01x04 J2
+U 1 1 5F44F858
+P 1350 5350
+F 0 "J2" H 1268 5667 50  0000 C CNN
+F 1 "Audio_In_Out" H 1268 5576 50  0000 C CNN
+F 2 "Connector_JST:JST_XH_B4B-XH-A_1x04_P2.50mm_Vertical" H 1350 5350 50  0001 C CNN
+F 3 "~" H 1350 5350 50  0001 C CNN
+	1    1350 5350
+	-1   0    0    -1
+$EndComp
+Text GLabel 1600 5450 2    59   Input ~ 0
+Audio_Out
+Wire Wire Line
+	1550 5350 2200 5350
+Wire Wire Line
+	1550 5250 2600 5250
+Wire Wire Line
+	1600 5450 1550 5450
+Wire Wire Line
+	1550 5550 2200 5550
+Connection ~ 2200 5550
+Wire Wire Line
+	2200 5550 2200 5700
 $EndSCHEMATC

Commit message: Update: PCB Design
Connections:
- net Audio_Out: now also J2.1 (Pin_1); no longer J2.3 (Pin_3)
- net GND: now also J2.3 (Pin_3); no longer J2.4 (Pin_4)
- net at RV1.3: now also J2.4 (Pin_4); no longer J2.1 (Pin_1)
Other:
- moved on the sheet: J2
Changed lines of the file:
@@
 	1    0    0    -1
 $EndComp
-Wire Wire Line
-	2200 5350 2200 5550
 $Comp
 L power:GND #PWR011
@@
 L Connector_Generic:Conn_01x04 J2
 U 1 1 5F44F858
-P 1350 5350
-F 0 "J2" H 1268 5667 50  0000 C CNN
-F 1 "Audio_In_Out" H 1268 5576 50  0000 C CNN
-F 2 "Connector_JST:JST_XH_B4B-XH-A_1x04_P2.50mm_Vertical" H 1350 5350 50  0001 C CNN
-F 3 "~" H 1350 5350 50  0001 C CNN
-	1    1350 5350
+P 1800 5050
+F 0 "J2" H 1718 5367 50  0000 C CNN
+F 1 "Audio_In_Out" H 1718 5276 50  0000 C CNN
+F 2 "Connector_JST:JST_XH_B4B-XH-A_1x04_P2.50mm_Vertical" H 1800 5050 50  0001 C CNN
+F 3 "~" H 1800 5050 50  0001 C CNN
+	1    1800 5050
 	-1   0    0    -1
 $EndComp
-Text GLabel 1600 5450 2    59   Input ~ 0
+Text GLabel 2100 4950 2    59   Input ~ 0
 Audio_Out
 Wire Wire Line
-	1550 5350 2200 5350
-Wire Wire Line
-	1550 5250 2600 5250
-Wire Wire Line
-	1600 5450 1550 5450
-Wire Wire Line
-	1550 5550 2200 5550
-Connection ~ 2200 5550
-Wire Wire Line
-	2200 5550 2200 5700
+	2000 4950 2100 4950
+Wire Wire Line
+	2000 5050 2200 5050
+Wire Wire Line
+	2200 5050 2200 5150
+Wire Wire Line
+	2600 5250 2000 5250
+Wire Wire Line
+	2000 5150 2200 5150
+Connection ~ 2200 5150
+Wire Wire Line
+	2200 5150 2200 5700
 $EndSCHEMATC
